Commit message: fixed intialization and swing control bug

File: resources/robots/pat/urdf/pat.urdf (robot description, URDF)
Before this commit: robot mini_cheetah_vision, 10 links, 9 joints
Links:
- link R_foot: mass None -> 0.06; geometry collision sphere radius=0.0185

Commit message: pat joint pd training

File: resources/robots/pat/urdf/pat.urdf (robot description, URDF)
Before this commit: robot mini_cheetah_vision, 10 links, 9 joints
Links:
- link L_thigh: geometry collision box size=0.2 0.0245 0.034; visual mesh filename=../meshes/thigh_l.dae scale=1 1 1
- link R_thigh: geometry collision box size=0.2 0.0245 0.034; visual mesh filename=../meshes/thigh_r.dae scale=1 1 1
- link trunk: geometry collision box size=0.10 0.18 0.25; visual mesh filename=../meshes/torso.dae scale=1 1 1

Commit message: update urdf

File: resources/robots/pat/urdf/pat.urdf (robot description, URDF)
Before this commit: robot mini_cheetah_vision, 10 links, 9 joints
Joints:
- joint L_hip_joint: origin xyz=0.0015 0.045 -0.06827 rpy=0 0 0 -> xyz=-0.0475 0.045 -0.06127 rpy=0 0 0
- joint R_hip_joint: origin xyz=0.0015 -0.045 -0.06827 rpy=0 0 0 -> xyz=-0.0475 -0.045 -0.06127 rpy=0 0 0

Commit message: sanity commit

File: resources/robots/pat/urdf/pat.urdf (robot description, URDF)
Before this commit: robot mini_cheetah_vision, 10 links, 9 joints
Links:
- link trunk: geometry collision box size=0.10 0.18 0.25; visual mesh filename=../meshes/body.dae scale=1 1 1
Joints:
- joint L_calf_joint: limit lower=-2.5 upper=1.5 effort=17 velocity=40 -> lower=-2.5 upper=1.5 effort=18 velocity=25
- joint L_hip_joint: limit lower=-0.8 upper=0.8 effort=17 velocity=40 -> lower=-0.8 upper=0.8 effort=9 velocity=40; origin xyz=0.0015 0.045 -0.06827 rpy=0 0 0 -> xyz=-0.047 0.045 -0.06827 rpy=0 0 0
- joint L_thigh_joint: limit lower=-1.5 upper=1.5 effort=17 velocity=40 -> lower=-1.5 upper=1.5 effort=18 velocity=25
- joint R_calf_joint: limit lower=-2.5 upper=1.5 effort=17 velocity=40 -> lower=-2.5 upper=1.5 effort=18 velocity=25
- joint R_hip_joint: limit lower=-0.8 upper=0.8 effort=17 velocity=40 -> lower=-0.8 upper=0.8 effort=9 velocity=40; origin xyz=0.0015 -0.045 -0.06827 rpy=0 0 0 -> xyz=-0.047 -0.045 -0.06827 rpy=0 0 0
- joint R_thigh_joint: limit lower=-1.5 upper=1.5 effort=17 velocity=40 -> lower=-1.5 upper=1.5 effort=18 velocity=25
